Commit message: code for thesis

File: rotors_description/urdf/component_snippets.xacro (robot description, xacro)
@@ -72,4 +72,5 @@
     <gazebo reference="${namespace}/camera_${camera_suffix}_link">
       <sensor type="camera" name="${namespace}_camera_${camera_suffix}">
+      <visualize>true</visualize>
         <update_rate>${frame_rate}</update_rate>
         <camera name="head">

File: rotors_description/urdf/iris_base.xacro (robot description, xacro)
@@ -10,4 +10,22 @@
     <xacro:default_mavlink_interface namespace="${namespace}" imu_sub_topic="imu" rotor_count="4" />
   </xacro:if>
+  <xacro:camera_macro
+    namespace="${namespace}"
+    parent_link="${namespace}/base_link"
+    camera_suffix="red_iris"
+    frame_rate="30.0"
+    horizontal_fov="1.3962634"
+    image_width="800"
+    image_height="800"
+    image_format="R8G8B8"
+    min_distance="0.02"
+    max_distance="300"
+    noise_mean="0.0"
+    noise_stddev="0.007"
+    enable_visual="true"
+    >
+  <box size="0.05 0.05 0.05" />
+  <origin xyz="0 0 -0.07" rpy="0 0.785398161 0"/>
+  </xacro:camera_macro>
   <!-- Mount an ADIS16448 IMU. -->
   <xacro:default_imu namespace="${namespace}" parent_link="${namespace}/base_link" />
